File: PCB/MainBoard/MainBoard.kicad_pcb (KiCad board)
At the start: 2 copper layers, 100 x 100 mm, 38 parts, among them CON1 BARREL_JACK, P1 PANTALLA, P10 CONN_01X02, P11 CONN_01X02, P12 DIP_SWITCH, P13 CONN_01X02, P14 CONN_01X02, P15 CONN_02X03, P16 CONN_RASPY, P19 IR_ARRAY, P2 REG_5V, P20 IR_SENSORS, P21 Reg_6V_IN, P22 CONN_RASPY, P24 CONN_01X24, P25 CONN_01X24, P28 Reg_6V_OUT, P3 SERVO_LIDAR, P32 CONN_01X02, P34 LEFT_ENCODER, P35 RIGHT_ENCODER, P4 MOTOR_DRIVER, P5 MOTOR_DRIVER, P6 CONN_01X03, P7 CONN_01X10, P8 SERVO_CLAW, P9 DIP_SWITCH, SW1 SWITCH_INV, SW3 SW_PUSH, SW4 SW_PUSH

Commit message: improving silks layers in PCB
Parts:
- D1: renamed from P1; value PANTALLA -> OLED DISPLAY
- J1 OPY: renamed from P16
- J2 AO_IR: renamed from P13
- J3 LF_IR: renamed from P14
- J4 ENC: renamed from P32
- P10: renamed from P19; value IR_ARRAY -> AO_IR
- P18: renamed from P8; value SERVO_CLAW -> SERVO_CLAMP
- P22: renamed from P7; value CONN_01X10 -> AO_IR | LW_IR
- P7: renamed from P9; value DIP_SWITCH -> DIP_SW
- REG1: renamed from P2; value REG_5V -> S7V7F5
- SW1: value SWITCH_INV -> OFF_SWITCH_ON
- renumbered C3 to C1, P4 to P1, P20 to P11, P22 to P12, P10 to P13, P21 to P14, P28 to P15, P34 to P16, P35 to P17, P3 to P19, P5 to P2, P6 to P20, P11 to P21, P24 to P4, P25 to P5, P12 to P8, P15 to P9, SW3 to SW2, SW4 to SW3
Other:
- board text added: "+"
- board text added: "-"
- board text added: "- GND -"
- board text added: "220"
- board text added: "22K"
- board text added: "BLUETOOTH"
- board text added: "LF_IR"
- board text added: "P3"
- board text added: "P6"
- board text added: "R1"
- board text added: "RX"
- board text added: "TX"
- board text added: "VM MD"
- board text added: "https://github.com/snailstorming/anedubot"
