File: PCB/MainBoard/MainBoard.kicad_pcb (KiCad board)
At the start: 2 copper layers, 100 x 100 mm, 38 parts, among them CON1 BARREL_JACK, J1 OPY CONN_RASPY, J2 AO_IR CONN_01X02, J3 LF_IR CONN_01X02, J4 ENC CONN_01X02, P1 MOTOR_DRIVER, P10 AO_IR, P11 IR_SENSORS, P12 CONN_RASPY, P13 CONN_01X02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

Commit message: Improving PCB silks layers
Other:
- outline, holes or cut-outs redrawn
- board text added: "A-SERVO"
- board text added: "RX TX O-PY"
Changed lines of the file:
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@@
   (general
     (links 106)
-    (no_connects 8)
-    (area 36.260389 36.260389 163.739611 163.739611)
+    (no_connects 2)
+    (area 49.924999 49.924999 150.075001 150.075001)
     (thickness 1.6)
-    (drawings 98)
+    (drawings 101)
     (tracks 324)
     (zones 0)
@@
     (0 F.Cu signal)
     (31 B.Cu signal)
-    (32 B.Adhes user)
-    (33 F.Adhes user)
-    (34 B.Paste user)
-    (35 F.Paste user)
+    (32 B.Adhes user hide)
+    (33 F.Adhes user hide)
+    (34 B.Paste user hide)
+    (35 F.Paste user hide)
     (36 B.SilkS user)
     (37 F.SilkS user)
@@
     (add_net +BATT)
   )
+  (module Pin_Headers:Pin_Header_Straight_1x02 (layer F.Cu)
+    (at 69.52 53.645 270)
+    (descr "Through hole pin header")
+    (tags "pin header")
+    (fp_text reference P13 (at 4.699 4.064 360) (layer B.SilkS)
+      (effects (font (size 1 1) (thickness 0.15)) (justify mirror))
+    )
+    (fp_text value CONN_01X02 (at -9.525 -4.064 270) (layer F.Fab)
+      (effects (font (size 1 1) (thickness 0.15)))
+    )
+    (fp_line (start -2.794 -2.032) (end -2.794 5.461) (layer B.SilkS) (width 0.15))
+    (fp_line (start 3.5 -2) (end -3.5 -2) (layer B.SilkS) (width 0.15))
+    (fp_line (start -3.5 -2) (end -3.5 5.5) (layer B.SilkS) (width 0.15))
+    (fp_line (start -3.5 5.5) (end 3.5 5.5) (layer B.SilkS) (width 0.15))
+    (fp_line (start 3.5 5.5) (end 3.5 -2) (layer B.SilkS) (width 0.15))
+    (fp_line (start -1.75 -1.75) (end -1.75 4.3) (layer F.CrtYd) (width 0.05))
+    (fp_line (start 1.75 -1.75) (end 1.75 4.3) (layer F.CrtYd) (width 0.05))
+    (fp_line (start -1.75 -1.75) (end 1.75 -1.75) (layer F.CrtYd) (width 0.05))
+    (fp_line (start -1.75 4.3) (end 1.75 4.3) (layer F.CrtYd) (width 0.05))
+    (pad 1 thru_hole rect (at 0 0 270) (size 2.3 2.3) (drill 1.2) (layers *.Cu *.Mask F.SilkS)
+      (net 1 GND))
+    (pad 2 thru_hole oval (at 0 3.5 270) (size 2.3 2.3) (drill 1.2) (layers *.Cu *.Mask F.SilkS)
+      (net 3 +BATT))
+    (model Pin_Headers.3dshapes/Pin_Header_Straight_1x02.wrl
+      (at (xyz 0 -0.05 0))
+      (scale (xyz 1 1 1))
+      (rotate (xyz 0 0 90))
+    )
+  )
   (module Pin_Headers:Pin_Header_Straight_2x02 (layer F.Cu)
     (at 132.14 128.55 270)
@@
     (fp_line (start 1.27 3.81) (end -1.27 3.81) (layer B.SilkS) (width 0.15))
     (fp_line (start -1.27 3.81) (end -1.27 -1.27) (layer B.SilkS) (width 0.15))
-    (fp_text user OPY (at 2.54 1.27 360) (layer F.SilkS)
+    (fp_text user OPY (at 2.4384 2.3114 360) (layer F.SilkS)
       (effects (font (size 1 1) (thickness 0.15)))
     )
@@
     (model Pin_Headers.3dshapes/Pin_Header_Straight_1x03.wrl
       (at (xyz 0 -0.1 0))
-      (scale (xyz 1 1 1))
-      (rotate (xyz 0 0 90))
-    )
-  )
-  (module Pin_Headers:Pin_Header_Straight_1x02 (layer F.Cu)
-    (at 69.52 53.645 270)
-    (descr "Through hole pin header")
-    (tags "pin header")
-    (fp_text reference P13 (at 4.699 4.064 360) (layer B.SilkS)
-      (effects (font (size 1 1) (thickness 0.15)) (justify mirror))
-    )
-    (fp_text value CONN_01X02 (at -9.525 -4.064 270) (layer F.Fab)
-      (effects (font (size 1 1) (thickness 0.15)))
-    )
-    (fp_line (start 3.5 -2) (end -3.5 -2) (layer B.SilkS) (width 0.15))
-    (fp_line (start -3.5 -2) (end -3.5 5.5) (layer B.SilkS) (width 0.15))
-    (fp_line (start -3.5 5.5) (end 3.5 5.5) (layer B.SilkS) (width 0.15))
-    (fp_line (start 3.5 5.5) (end 3.5 -2) (layer B.SilkS) (width 0.15))
-    (fp_line (start -1.75 -1.75) (end -1.75 4.3) (layer F.CrtYd) (width 0.05))
-    (fp_line (start 1.75 -1.75) (end 1.75 4.3) (layer F.CrtYd) (width 0.05))
-    (fp_line (start -1.75 -1.75) (end 1.75 -1.75) (layer F.CrtYd) (width 0.05))
-    (fp_line (start -1.75 4.3) (end 1.75 4.3) (layer F.CrtYd) (width 0.05))
-    (pad 1 thru_hole rect (at 0 0 270) (size 2.3 2.3) (drill 1.2) (layers *.Cu *.Mask F.SilkS)
-      (net 1 GND))
-    (pad 2 thru_hole oval (at 0 3.5 270) (size 2.3 2.3) (drill 1.2) (layers *.Cu *.Mask F.SilkS)
-      (net 3 +BATT))
-    (model Pin_Headers.3dshapes/Pin_Header_Straight_1x02.wrl
-      (at (xyz 0 -0.05 0))
       (scale (xyz 1 1 1))
       (rotate (xyz 0 0 90))
@@
       (net 4 "Net-(D2-Pad2)"))
   )
+  (gr_text A-SERVO (at 78.283 110.9728 90) (layer F.SilkS)
+    (effects (font (size 1 1) (thickness 0.15)))
+  )
+  (gr_text "RX TX\nO-PY" (at 78.9434 127.8892 90) (layer F.SilkS)
+    (effects (font (size 1 1) (thickness 0.15)))
+  )
+  (gr_text + (at 65.964 56.312) (layer F.SilkS)
+    (effects (font (size 1.5 1.5) (thickness 0.25)))
+  )
+  (gr_text - (at 69.52 56.312) (layer F.SilkS)
+    (effects (font (size 1.5 1.5) (thickness 0.25)))
+  )
   (gr_text "VM MD" (at 85.268 126.416 270) (layer F.SilkS)
     (effects (font (size 1 1) (thickness 0.15)))
@@
   (gr_line (start 140.5 50) (end 150 59.5) (angle 90) (layer Edge.Cuts) (width 0.15))
   (gr_line (start 139.25 50) (end 140.5 50) (angle 90) (layer Edge.Cuts) (width 0.15))
-  (gr_line (start 50 59.75) (end 50 59.5) (angle 90) (layer Edge.Cuts) (width 0.15))
   (gr_circle (center 100 100) (end 55 55) (layer Cmts.User) (width 0.2))
   (gr_line (start 132.15 100) (end 137.23 100) (angle 90) (layer Cmts.User) (width 0.2))
